File: pcb/switch_matrix.kicad_sch (KiCad schematic)
At the start: 21 parts, among them U1 SN74LVC1G139, U2 TLP161J, U3 TLP161J, U4 TLP161J, U5 TLP161J, U6 TLP161J, U7 TLP161J

Commit message: WiP battery management
Parts:
- C5: value 10uF -> 4.7uF
Changed lines of the file:
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@@
       (effects (font (size 1.27 1.27)) (justify left))
     )
-    (property "Value" "10uF" (at 218.44 97.79 0)
+    (property "Value" "4.7uF" (at 218.44 97.79 0)
       (effects (font (size 1.27 1.27)) (justify left))
     )
