File: pcb/power_management.kicad_sch (KiCad schematic)
At the start: 18 parts, among them U10 MCP73831-2-OT, U11 HT7530-1, U12 HX3608

Commit message: Notes
Other:
- note added: "FIXME: Think MCU Cheapo STM32 for everyone to use or monolithic system"
Changed lines of the file:
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@@
+    (effects (font (size 1.27 1.27)) (justify left bottom))
+  )
+  (text "FIXME: Think MCU\nCheapo STM32 for \neveryone to use or \nmonolithic system"
+    (at 80.01 60.96 0)
     (effects (font (size 1.27 1.27)) (justify left bottom))
   )
